File: motherboard/motherboard.brd (EAGLE design)
At the start: 100.3 x 100.3 mm, 136 parts, among them IC1 TL074D, IC2 TL074D, IC3 TL074D, IC4 78L05, IC5 78L33, J1 JACK_3.5MMPJ301BM, J10 JACK_3.5MMPJ301BM, J11 JACK_3.5MMPJ301BM, J2 JACK_3.5MMPJ301BM, J3 JACK_3.5MMPJ301BM, J4 JACK_3.5MMPJ301BM, J5 JACK_3.5MMPJ301BM, J6 JACK_3.5MMPJ301BM, J7 JACK_3.5MMPJ301BM, J8 JACK_3.5MMPJ301BM, J9 JACK_3.5MMPJ301BM, Q1 2N3904, U1 TL074D, U2 TL074D

Commit message: Adjust layout
Parts:
- removed IC3: TL074D, linear:SO14
- removed IC4: 78L05, linear:TO92
- removed IC5: 78L33, linear:TO92
- removed OK1, OK2: VTL5C, optocoupler:VTL5C
- added U3, U4, U5: OP_QUAD_SMD, kweiwen:SO14
- added V1, V2: VACTROL, kweiwen:VACTROL_4PIN_VTL5C
- C22: value (none) -> 100n
- D9: value (none) -> 3mm
- IC1: value TL074D -> 78L05; device linear:SO14 -> linear:TO92
- IC2: value TL074D -> 78L33; device linear:SO14 -> linear:TO92
- U1, U2: value TL074D -> OP_QUAD_SMD
- moved U1 61.6 mm to (82.5, 55.2), turned to 90 degrees
- moved IC1 54.2 mm to (34.3, 80.0), turned to 0 degrees
- moved U2 32.9 mm to (49.5, 55.2), turned to 90 degrees
- moved IC2 31.2 mm to (68.6, 80.0), turned to 0 degrees
- moved C20 7.28 mm to (58.7, 20.3), turned to 0 degrees
- moved C21 2.16 mm to (58.7, 14.0)
- moved R47 1.14 mm to (80.1, 14.0), flipped to the top
- renumbered LED1 to D9
Connections:
- net +12V: now also IC1.3, IC2.3, U3.4, U4.4, U5.4, V1.2, V2.2; no longer IC1.4, IC2.4, IC3.4, IC4.3, IC5.3, OK1.2, OK2.2
- net +3.3V: now also IC2.1; no longer IC5.1
- net +5V: now also IC1.1; no longer IC4.1
- net -12V: now also U3.11, U4.11, U5.11; no longer IC1.11, IC2.11, IC3.11
- net COLLECTOR: now also V1.1, V2.1; no longer OK1.1, OK2.1
- net GND: now also IC1.2, IC2.2, U2.3, U2.5, U3.10, U3.12, U3.3, U3.5, U4.10, U4.12, U4.3, U4.5, U5.10, U5.12; no longer IC1.10, IC1.12, IC1.3, IC1.5, IC2.10, IC2.12, IC2.3, IC2.5, IC3.10, IC3.12, IC3.3, IC3.5, IC4.2, IC5.2
- net N$11: now also U1.13; no longer IC1.13
- net N$12: now also U1.14; no longer IC1.14
- net N$14: now also U5.8; no longer U2.8
- net N$16: now also U5.13; no longer U2.13
- net N$17: now also U5.14; no longer U2.14
- net N$18: now also U5.9; no longer U2.9
- net N$19: now also U2.9; no longer IC2.9
- net N$20: now also U2.8; no longer IC2.8
- net N$21: now also U2.13; no longer IC2.13
- net N$22: now also U2.14; no longer IC2.14
- net N$25: now also U2.6; no longer IC2.6
- net N$26: now also U2.7; no longer IC2.7
- net N$27: now also U2.2; no longer IC2.2
- net N$28: now also U2.1; no longer IC2.1
- net N$3: now also U1.6; no longer IC1.6
- net N$30: now also U5.6; no longer U2.6
- net N$33: now also U3.9; no longer IC3.9
- net N$34: now also U3.8; no longer IC3.8
- net N$35: now also U3.13; no longer IC3.13
- net N$36: now also U3.14; no longer IC3.14
- net N$39: now also U3.6; no longer IC3.6
- net N$4: now also U1.7; no longer IC1.7
- net N$40: now also U3.7; no longer IC3.7
- net N$41: now also U3.2; no longer IC3.2
- net N$42: now also U3.1; no longer IC3.1
- net N$45: now also U5.7; no longer U2.7
- net N$46: now also U5.5, V1.4; no longer OK1.3, U2.5
- net N$5: now also U1.2; no longer IC1.2
- net N$53: now also U5.2; no longer U2.2
- net N$54: now also U5.1; no longer U2.1
- net N$55: now also U5.3, V2.4; no longer OK2.3, U2.3
- net N$6: now also U1.1; no longer IC1.1
- net N$69: now also U4.13; no longer U1.13
- net N$70: now also U4.14; no longer U1.14
- net N$72: now also U4.9; no longer U1.9
- net N$73: now also U4.8; no longer U1.8
- net N$74: now also U4.1; no longer U1.1
- net N$75: now also U4.7; no longer U1.7
- net N$78: now also U4.2; no longer U1.2
- net N$79: now also U4.6; no longer U1.6
- net N$8: now also U1.9; no longer IC1.9
- net N$9: now also U1.8; no longer IC1.8
- net WET_L: now also V1.3; no longer OK1.4
- net WET_R: now also V2.3; no longer OK2.4
Routing:
- net GND: track 1004.4 -> 1019.1 mm
- net N$55: track 28.0 -> 21.1 mm
- net +12V: track 393.6 -> 400.2 mm
- net N$46: track 51.0 -> 45.1 mm, vias 1 -> 0
- net WET_R: track 26.2 -> 22.4 mm
- net -12V: track 333.4 -> 329.6 mm
- net N$13: track 23.2 -> 20.0 mm
- net N$24: track 28.7 -> 26.6 mm
- net N$48: track 6.79 -> 5.40 mm
- net COLLECTOR: track 38.4 -> 39.5 mm
