File: motherboard/motherboard.sch (EAGLE design)
At the start: 136 parts, among them IC1 TL074D, IC2 TL074D, IC3 TL074D, IC4 78L05, IC5 78L33, J1 JACK_3.5MMPJ301BM, J10 JACK_3.5MMPJ301BM, J11 JACK_3.5MMPJ301BM, J2 JACK_3.5MMPJ301BM, J3 JACK_3.5MMPJ301BM, J4 JACK_3.5MMPJ301BM, J5 JACK_3.5MMPJ301BM, J6 JACK_3.5MMPJ301BM, J7 JACK_3.5MMPJ301BM, J8 JACK_3.5MMPJ301BM, J9 JACK_3.5MMPJ301BM, Q1 2N3904, U1 TL074D, U2 TL074D

Commit message: Adjust layout
Parts:
- removed IC3: TL074D, linear:TL074D
- removed IC4: 78L05, linear:78L05Z
- removed IC5: 78L33, linear:78L05Z
- removed LED1: (no value), led:LED3MM
- removed OK1, OK2: VTL5C, optocoupler:VTL5C
- added D9: 3mm, led:LED3MM
- added U3, U4, U5: OP_QUAD_SMD, kweiwen:OP_QUAD_SMD
- added V1, V2: VACTROL, kweiwen:VACTROL
- C22: value (none) -> 100n
- IC1: value TL074D -> 78L05; device linear:TL074D -> linear:78L05Z
- IC2: value TL074D -> 78L33; device linear:TL074D -> linear:78L05Z
- U1, U2: value TL074D -> OP_QUAD_SMD; device kweiwen:TL074D -> kweiwen:OP_QUAD_SMD
Connections:
- net +12V: now also IC1.VI, IC2.VI, U3P.V+, U4P.V+, U5P.V+, V1.LED+, V2.LED+; no longer IC1P.V+, IC2P.V+, IC3P.V+, IC4.VI, IC5.VI, OK1.2, OK2.2
- net +3.3V: now also D1.C2, D2.C2, D3.C2, D4.C2, D5.C2, D6.C2, IC2.VO; no longer D1.C, D2.C, D3.C, D4.C, D5.C, D6.C, IC5.VO
- net +5V: now also IC1.VO; no longer IC4.VO
- net -12V: now also U3P.V-, U4P.V-, U5P.V-; no longer IC1P.V-, IC2P.V-, IC3P.V-
- net CH1: now also D1.C1A2; no longer D1.CA
- net CH2: now also D2.C1A2; no longer D2.CA
- net CH3: now also D3.C1A2; no longer D3.CA
- net CH4: now also D4.C1A2; no longer D4.CA
- net CH5: now also D5.C1A2; no longer D5.CA
- net CH6: now also D6.C1A2; no longer D6.CA
- net COLLECTOR: now also V1.LED-, V2.LED-; no longer OK1.1, OK2.1
- net GND: now also D1.A1, D2.A1, D3.A1, D4.A1, D5.A1, D6.A1, D9.C, IC1.GND, IC2.GND, U2A.+IN, U2B.+IN, U3A.+IN, U3B.+IN, U3C.+IN, U3D.+IN, U4A.+IN, U4B.+IN, U4C.+IN, U4D.+IN, U5C.+IN, U5D.+IN; no longer D1.A, D2.A, D3.A, D4.A, D5.A, D6.A, IC1A.+IN, IC1B.+IN, IC1C.+IN, IC1D.+IN, IC2A.+IN, IC2B.+IN, IC2C.+IN, IC2D.+IN, IC3A.+IN, IC3B.+IN, IC3C.+IN, IC3D.+IN, IC4.GND, IC5.GND, LED1.C
- net N$11: now also U1D.-IN; no longer IC1D.-IN
- net N$12: now also U1D.OUT; no longer IC1D.OUT
- net N$14: now also U5C.OUT; no longer U2C.OUT
- net N$16: now also U5D.-IN; no longer U2D.-IN
- net N$17: now also U5D.OUT; no longer U2D.OUT
- net N$18: now also U5C.-IN; no longer U2C.-IN
- net N$19: now also U2C.-IN; no longer IC2C.-IN
- net N$20: now also U2C.OUT; no longer IC2C.OUT
- net N$21: now also U2D.-IN; no longer IC2D.-IN
- net N$22: now also U2D.OUT; no longer IC2D.OUT
- net N$25: now also U2B.-IN; no longer IC2B.-IN
- net N$26: now also U2B.OUT; no longer IC2B.OUT
- net N$27: now also U2A.-IN; no longer IC2A.-IN
- net N$28: now also U2A.OUT; no longer IC2A.OUT
- net N$29: now also D9.A; no longer LED1.A
- net N$3: now also U1B.-IN; no longer IC1B.-IN
- net N$30: now also U5B.-IN; no longer U2B.-IN
- net N$33: now also U3C.-IN; no longer IC3C.-IN
- net N$34: now also U3C.OUT; no longer IC3C.OUT
- net N$35: now also U3D.-IN; no longer IC3D.-IN
- net N$36: now also U3D.OUT; no longer IC3D.OUT
- net N$39: now also U3B.-IN; no longer IC3B.-IN
- net N$4: now also U1B.OUT; no longer IC1B.OUT
- net N$40: now also U3B.OUT; no longer IC3B.OUT
- net N$41: now also U3A.-IN; no longer IC3A.-IN
- net N$42: now also U3A.OUT; no longer IC3A.OUT
- net N$45: now also U5B.OUT; no longer U2B.OUT
- net N$46: now also U5B.+IN, V1.RES2; no longer OK1.3, U2B.+IN
- net N$5: now also U1A.-IN; no longer IC1A.-IN
- net N$53: now also U5A.-IN; no longer U2A.-IN
- net N$54: now also U5A.OUT; no longer U2A.OUT
- net N$55: now also U5A.+IN, V2.RES2; no longer OK2.3, U2A.+IN
- net N$6: now also U1A.OUT; no longer IC1A.OUT
- net N$69: now also U4D.-IN; no longer U1D.-IN
- net N$70: now also U4D.OUT; no longer U1D.OUT
- net N$72: now also U4C.-IN; no longer U1C.-IN
- net N$73: now also U4C.OUT; no longer U1C.OUT
- net N$74: now also U4A.OUT; no longer U1A.OUT
- net N$75: now also U4B.OUT; no longer U1B.OUT
- net N$78: now also U4A.-IN; no longer U1A.-IN
- net N$79: now also U4B.-IN; no longer U1B.-IN
- net N$8: now also U1C.-IN; no longer IC1C.-IN
- net N$9: now also U1C.OUT; no longer IC1C.OUT
- net WET_L: now also V1.RES1; no longer OK1.4
- net WET_R: now also V2.RES1; no longer OK2.4
Other:
- moved on the sheet: C13, C14, C15, C16, C17, C18, C19, C20, C21, J10, J11, J7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
