File: hardware/mother/mother.brd (EAGLE design)
At the start: 100.3 x 100.3 mm, 136 parts, among them IC1 78L05, IC2 78L33, J1 JACK_3.5MMPJ301BM, J10 JACK_3.5MMPJ301BM, J11 JACK_3.5MMPJ301BM, J2 JACK_3.5MMPJ301BM, J3 JACK_3.5MMPJ301BM, J4 JACK_3.5MMPJ301BM, J5 JACK_3.5MMPJ301BM, J6 JACK_3.5MMPJ301BM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

Commit message: SPDT ON-ON
Parts:
- VR8: value (none) -> 50k
Other:
- board text added: "designed & assembled in tainan, taiwan. 2017"
Changed lines of the file:
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@@
 <layer number="23" name="tOrigins" color="15" fill="1" visible="yes" active="yes"/>
 <layer number="24" name="bOrigins" color="15" fill="1" visible="yes" active="yes"/>
-<layer number="25" name="tNames" color="7" fill="1" visible="yes" active="yes"/>
+<layer number="25" name="tNames" color="7" fill="1" visible="no" active="yes"/>
 <layer number="26" name="bNames" color="7" fill="1" visible="no" active="yes"/>
 <layer number="27" name="tValues" color="7" fill="1" visible="no" active="yes"/>
@@
 <text x="51.435" y="5.08" size="1.2192" layer="22" ratio="12" rot="MR270" align="center">Red
 Stripe!</text>
+<text x="69.215" y="40.005" size="1.905" layer="22" font="fixed" ratio="16" rot="MR180" align="center">designed &amp; assembled in
+tainan, taiwan. 2017</text>
 </plain>
 <attributes>
@@
 </element>
 <element name="C14" library="eagle-ltspice" package="C0603" value="220p" x="66.3575" y="24.765" smashed="yes" rot="R270">
-<attribute name="NAME" x="64.3255" y="24.765" size="1.27" layer="25" rot="R270"/>
+<attribute name="NAME" x="64.5795" y="24.765" size="1.016" layer="25" rot="R270"/>
 <attribute name="SPICEMODEL" value="NONE" x="66.3575" y="24.765" size="1.778" layer="27" rot="R270" display="off"/>
 <attribute name="SPICEPREFIX" value="C" x="66.3575" y="24.765" size="1.778" layer="27" rot="R270" display="off"/>
@@
 </element>
 <element name="C15" library="eagle-ltspice" package="C0603" value="220p" x="75.8825" y="24.765" smashed="yes" rot="R270">
-<attribute name="NAME" x="76.7715" y="24.765" size="1.27" layer="25" rot="R270"/>
+<attribute name="NAME" x="76.7715" y="24.765" size="1.016" layer="25" rot="R270"/>
 <attribute name="SPICEMODEL" value="NONE" x="75.8825" y="24.765" size="1.778" layer="27" rot="R270" display="off"/>
 <attribute name="SPICEPREFIX" value="C" x="75.8825" y="24.765" size="1.778" layer="27" rot="R270" display="off"/>
@@
 </element>
 <element name="C16" library="eagle-ltspice" package="C0603" value="18p" x="33.3629" y="32.639" smashed="yes">
-<attribute name="NAME" x="36.068" y="32.2453" size="1.27" layer="25" rot="R90"/>
+<attribute name="NAME" x="36.068" y="32.2453" size="1.016" layer="25" rot="R90"/>
 <attribute name="SPICEMODEL" value="NONE" x="33.3629" y="32.639" size="1.778" layer="27" display="off"/>
 <attribute name="SPICEPREFIX" value="C" x="33.3629" y="32.639" size="1.778" layer="27" display="off"/>
@@
 </element>
 <element name="C17" library="eagle-ltspice" package="C0603" value="18p" x="19.9771" y="32.639" smashed="yes" rot="R180">
-<attribute name="NAME" x="18.4531" y="32.639" size="1.27" layer="25" rot="R180"/>
+<attribute name="NAME" x="18.4531" y="32.639" size="1.016" layer="25" rot="R180"/>
 <attribute name="SPICEMODEL" value="NONE" x="19.9771" y="32.639" size="1.778" layer="27" rot="R180" display="off"/>
 <attribute name="SPICEPREFIX" value="C" x="19.9771" y="32.639" size="1.778" layer="27" rot="R180" display="off"/>
@@
 </element>
 <element name="R31" library="eagle-ltspice" package="R0603" value="22k" x="22.987" y="23.495" smashed="yes" rot="R270">
-<attribute name="NAME" x="24.511" y="22.352" size="0.8128" layer="25" rot="R180"/>
+<attribute name="NAME" x="24.892" y="22.098" size="0.8128" layer="25" rot="R180"/>
 <attribute name="SPICEMODEL" value="NONE" x="22.987" y="23.495" size="1.778" layer="27" rot="R270" display="off"/>
 <attribute name="SPICEPREFIX" value="R" x="22.987" y="23.495" size="1.778" layer="27" rot="R270" display="off"/>
@@
 </element>
 <element name="R32" library="eagle-ltspice" package="R0603" value="22k" x="30.353" y="23.495" smashed="yes" rot="R270">
-<attribute name="NAME" x="31.369" y="22.352" size="0.8128" layer="25" rot="R180"/>
+<attribute name="NAME" x="30.48" y="22.098" size="0.8128" layer="25" rot="R180"/>
 <attribute name="SPICEMODEL" value="NONE" x="30.353" y="23.495" size="1.778" layer="27" rot="R270" display="off"/>
 <attribute name="SPICEPREFIX" value="R" x="30.353" y="23.495" size="1.778" layer="27" rot="R270" display="off"/>
@@
 </element>
 <element name="R34" library="eagle-ltspice" package="R0603" value="3.3k" x="25.019" y="23.495" smashed="yes" rot="R90">
-<attribute name="NAME" x="26.797" y="22.352" size="0.8128" layer="25" rot="R180"/>
+<attribute name="NAME" x="25.781" y="24.638" size="0.8128" layer="25" rot="R270"/>
 <attribute name="SPICEMODEL" value="NONE" x="25.019" y="23.495" size="1.778" layer="27" rot="R90" display="off"/>
 <attribute name="SPICEPREFIX" value="R" x="25.019" y="23.495" size="1.778" layer="27" rot="R90" display="off"/>
@@
 </element>
 <element name="R35" library="eagle-ltspice" package="R0603" value="3.3k" x="28.321" y="23.495" smashed="yes" rot="R90">
-<attribute name="NAME" x="29.083" y="22.352" size="0.8128" layer="25" rot="R180"/>
+<attribute name="NAME" x="26.797" y="24.638" size="0.8128" layer="25" rot="R270"/>
 <attribute name="SPICEMODEL" value="NONE" x="28.321" y="23.495" size="1.778" layer="27" rot="R90" display="off"/>
 <attribute name="SPICEPREFIX" value="R" x="28.321" y="23.495" size="1.778" layer="27" rot="R90" display="off"/>
@@
 </element>
 <element name="R38" library="eagle-ltspice" package="R0603" value="5.6k" x="20.955" y="23.495" smashed="yes" rot="R90">
-<attribute name="NAME" x="22.225" y="22.352" size="0.8128" layer="25" rot="R180"/>
+<attribute name="NAME" x="22.606" y="22.098" size="0.8128" layer="25" rot="R180"/>
 <attribute name="SPICEMODEL" value="NONE" x="20.955" y="23.495" size="1.778" layer="27" rot="R90" display="off"/>
 <attribute name="SPICEPREFIX" value="R" x="20.955" y="23.495" size="1.778" layer="27" rot="R90" display="off"/>
@@
 </element>
 <element name="R39" library="eagle-ltspice" package="R0603" value="5.6k" x="32.385" y="23.495" smashed="yes" rot="R90">
-<attribute name="NAME" x="33.655" y="22.352" size="0.8128" layer="25" rot="R180"/>
+<attribute name="NAME" x="32.766" y="22.098" size="0.8128" layer="25" rot="R180"/>
 <attribute name="SPICEMODEL" value="NONE" x="32.385" y="23.495" size="1.778" layer="27" rot="R90" display="off"/>
 <attribute name="SPICEPREFIX" value="R" x="32.385" y="23.495" size="1.778" layer="27" rot="R90" display="off"/>
@@
 </element>
 <element name="R41" library="eagle-ltspice" package="R0603" value="5.6k" x="18.923" y="23.495" smashed="yes" rot="R270">
-<attribute name="NAME" x="19.939" y="22.352" size="0.8128" layer="25" rot="R180"/>
+<attribute name="NAME" x="20.32" y="22.098" size="0.8128" layer="25" rot="R180"/>
 <attribute name="SPICEMODEL" value="NONE" x="18.923" y="23.495" size="1.778" layer="27" rot="R270" display="off"/>
 <attribute name="SPICEPREFIX" value="R" x="18.923" y="23.495" size="1.778" layer="27" rot="R270" display="off"/>
@@
 </element>
 <element name="R42" library="eagle-ltspice" package="R0603" value="5.6k" x="34.417" y="23.495" smashed="yes" rot="R270">
-<attribute name="NAME" x="35.941" y="22.352" size="0.8128" layer="25" rot="R180"/>
+<attribute name="NAME" x="35.052" y="22.098" size="0.8128" layer="25" rot="R180"/>
 <attribute name="SPICEMODEL" value="NONE" x="34.417" y="23.495" size="1.778" layer="27" rot="R270" display="off"/>
 <attribute name="SPICEPREFIX" value="R" x="34.417" y="23.495" size="1.778" layer="27" rot="R270" display="off"/>
@@
 </element>
 <element name="R52" library="eagle-ltspice" package="R0603" value="39k" x="33.3629" y="30.607" smashed="yes" rot="R180">
-<attribute name="NAME" x="36.068" y="27.6479" size="1.27" layer="25" rot="R90"/>
+<attribute name="NAME" x="36.068" y="28.9179" size="1.016" layer="25" rot="R90"/>
 <attribute name="SPICEMODEL" value="NONE" x="33.3629" y="30.607" size="1.778" layer="27" rot="R180" display="off"/>
 <attribute name="SPICEPREFIX" value="R" x="33.3629" y="30.607" size="1.778" layer="27" rot="R180" display="off"/>
@@
 </element>
 <element name="R53" library="eagle-ltspice" package="R0603" value="39k" x="19.9771" y="30.607" smashed="yes">
-<attribute name="NAME" x="18.4531" y="30.607" size="1.27" layer="25" rot="R180"/>
+<attribute name="NAME" x="18.4531" y="30.607" size="1.016" layer="25" rot="R180"/>
 <attribute name="SPICEMODEL" value="NONE" x="19.9771" y="30.607" size="1.778" layer="27" display="off"/>
 <attribute name="SPICEPREFIX" value="R" x="19.9771" y="30.607" size="1.778" layer="27" display="off"/>
@@
 </element>
 <element name="R58" library="eagle-ltspice" package="R0603" value="1k" x="77.47" y="27.9146" smashed="yes">
-<attribute name="NAME" x="76.2" y="28.5496" size="1.27" layer="25"/>
+<attribute name="NAME" x="76.2" y="28.6766" size="1.016" layer="25"/>
 <attribute name="SPICEMODEL" value="NONE" x="77.47" y="27.9146" size="1.778" layer="27" display="off"/>
 <attribute name="SPICEPREFIX" value="R" x="77.47" y="27.9146" size="1.778" layer="27" display="off"/>
@@
 </element>
 <element name="R59" library="eagle-ltspice" package="R0603" value="1k" x="64.77" y="27.9146" smashed="yes" rot="R180">
-<attribute name="NAME" x="66.04" y="27.2796" size="1.27" layer="25" rot="R180"/>
+<attribute name="NAME" x="66.04" y="27.1526" size="1.016" layer="25" rot="R180"/>
 <attribute name="SPICEMODEL" value="NONE" x="64.77" y="27.9146" size="1.778" layer="27" rot="R180" display="off"/>
 <attribute name="SPICEPREFIX" value="R" x="64.77" y="27.9146" size="1.778" layer="27" rot="R180" display="off"/>
@@
 <element name="D9" library="led" package="LED3MM" value="3mm" x="71.12" y="3.175" rot="R180"/>
 <element name="R43" library="kweiwen" package="1/4W_RESISTOR" value="" x="80.645" y="27.94" rot="R270"/>
-<element name="VR8" library="kweiwen" package="POT-DUAL-PTH-PANASONIC-VERT-KIT" value="" x="26.67" y="13.97" smashed="yes" rot="R270">
+<element name="VR8" library="kweiwen" package="POT-DUAL-PTH-PANASONIC-VERT-KIT" value="50k" x="26.67" y="13.97" smashed="yes" rot="R270">
 <attribute name="NAME" x="26.67" y="9.017" size="1.016" layer="25" font="vector" ratio="12" align="bottom-center"/>
 <attribute name="PROD_ID" value="RES-11897" x="26.67" y="13.97" size="1.778" layer="27" rot="R270" display="off"/>
