File: hardware/mother/mother.sch (EAGLE design)
At the start: 136 parts, among them IC1 78L05, IC2 78L33, J1 JACK_3.5MMPJ301BM, J10 JACK_3.5MMPJ301BM, J11 JACK_3.5MMPJ301BM, J2 JACK_3.5MMPJ301BM, J3 JACK_3.5MMPJ301BM, J4 JACK_3.5MMPJ301BM, J5 JACK_3.5MMPJ301BM, J6 JACK_3.5MMPJ301BM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

Commit message: Revert "Update"
This reverts commit 1fa1ac1b62750ae01fc9ebf9e2e8e41934c85bca, reversing
changes made to 5a165f026fc5e219df6fc06eabf06e676fb6696f.
Parts:
- C16, C17: value 1n -> 18p
- R43: value 330 -> (none)
- R45: value 147 -> 300
- R47: value 100 -> 1k
- R48, R49: value 56k -> (none)
- R52, R53: value 22K -> 39k
Changed lines of the file:
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@@
 <part name="C15" library="eagle-ltspice" deviceset="C" device="C0603" value="220p"/>
 <part name="GND51" library="SparkFun" deviceset="GND" device=""/>
-<part name="R49" library="eagle-ltspice" deviceset="R" device="R0603" value="56k"/>
+<part name="R49" library="eagle-ltspice" deviceset="R" device="R0603"/>
 <part name="GND54" library="SparkFun" deviceset="GND" device=""/>
 <part name="R51" library="eagle-ltspice" deviceset="R" device="R0603" value="5.6k"/>
 <part name="GND56" library="SparkFun" deviceset="GND" device=""/>
-<part name="R53" library="eagle-ltspice" deviceset="R" device="R0603" value="22K"/>
-<part name="C17" library="eagle-ltspice" deviceset="C" device="C0603" value="1n"/>
-<part name="R48" library="eagle-ltspice" deviceset="R" device="R0603" value="56k"/>
+<part name="R53" library="eagle-ltspice" deviceset="R" device="R0603" value="39k"/>
+<part name="C17" library="eagle-ltspice" deviceset="C" device="C0603" value="18p"/>
+<part name="R48" library="eagle-ltspice" deviceset="R" device="R0603"/>
 <part name="GND53" library="SparkFun" deviceset="GND" device=""/>
 <part name="R50" library="eagle-ltspice" deviceset="R" device="R0603" value="5.6k"/>
 <part name="GND55" library="SparkFun" deviceset="GND" device=""/>
-<part name="R52" library="eagle-ltspice" deviceset="R" device="R0603" value="22K"/>
-<part name="C16" library="eagle-ltspice" deviceset="C" device="C0603" value="1n"/>
+<part name="R52" library="eagle-ltspice" deviceset="R" device="R0603" value="39k"/>
+<part name="C16" library="eagle-ltspice" deviceset="C" device="C0603" value="18p"/>
 <part name="R56" library="eagle-ltspice" deviceset="R" device="R0603" value="1k"/>
 <part name="R34" library="eagle-ltspice" deviceset="R" device="R0603" value="3.3k"/>
@@
 <part name="GND58" library="SparkFun" deviceset="GND" device=""/>
 <part name="R46" library="eagle-ltspice" deviceset="R" device="R0603" value="200"/>
-<part name="R47" library="RepRapjr" deviceset="R-TRIMM" device="64W" value="100"/>
+<part name="R47" library="RepRapjr" deviceset="R-TRIMM" device="64W" value="1k"/>
 <part name="J9" library="kweiwen" deviceset="JACK_3.5MM" device="PJ301BM"/>
 <part name="J7" library="kweiwen" deviceset="JACK_3.5MM" device="PJ301BM"/>
@@
 <part name="GND71" library="SparkFun" deviceset="GND" device=""/>
 <part name="GND72" library="SparkFun" deviceset="GND" device=""/>
-<part name="R45" library="kweiwen" deviceset="*RESISTOR*" device="10MM" value="147"/>
+<part name="R45" library="kweiwen" deviceset="*RESISTOR*" device="10MM" value="300"/>
 <part name="D9" library="led" deviceset="LED" device="3MM" value="3mm"/>
-<part name="R43" library="kweiwen" deviceset="*RESISTOR*" device="10MM" value="330"/>
+<part name="R43" library="kweiwen" deviceset="*RESISTOR*" device="10MM"/>
 <part name="GND49" library="SparkFun" deviceset="GND" device=""/>
 <part name="VR8" library="kweiwen" deviceset="POTENTIOMETER_DUAL" device="-PTH-12MM-1/20W-20%-KIT" value="50k"/>
